File: hardware/mouse.kicad_pcb (KiCad board)
At the start: 4 copper layers, 44 x 68 mm, 88 parts, among them J2 JSTPH, J3 USB_C_Receptacle_USB2.0_14P, SW1 SW_SPST, SW2 SW_SPST, SW3 SW_SPST, SW4 SW_SPST, SW5 SW_SPST, SW6 SW_SPST, SW7 SW_SPST, SW8 RotaryEncoder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

Commit message: mostly just eod stuff, a couple csv files and readme changes
Parts:
- A1: value PAW3395 -> ~
Changed lines of the file:
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@@
 		(sheetname "/RF_Radio/")
 		(sheetfile "rfradio.kicad_sch")
-		(attr smd)
+		(attr smd dnp)
 		(fp_line
 			(start -0.261252 -0.735)
@@
 			)
 		)
-		(property "Value" "PAW3395"
+		(property "Value" "~"
 			(at 5.35 13.375 0)
 			(layer "F.Fab")
@@
 		(sheetname "/RF_Radio/")
 		(sheetfile "rfradio.kicad_sch")
-		(attr smd)
+		(attr smd dnp)
 		(fp_line
 			(start -0.261252 -0.735)
