File: hardware/mouse/_autosave-mouse.kicad_pcb (KiCad board)
At the start: 4 copper layers, 44 x 68 mm, 88 parts, among them J2 JSTPH, J3 USB_C_Receptacle_USB2.0_14P, SW1 SW_SPST, SW2 SW_SPST, SW3 SW_SPST, SW4 SW_SPST, SW5 SW_SPST, SW6 SW_SPST, SW7 SW_SPST, SW8 RotaryEncoder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

Commit message: added case v1
Routing:
- net C1-1: track 11.7 -> 14.1 mm
- net +BATT: track 108.4 -> 110.3 mm
- net D-: track 35.3 -> 36.7 mm
- net VDDW1: track 103.8 -> 104.9 mm
- net RECW: track 41.0 -> 40.2 mm
- net RECCW: track 37.2 -> 36.4 mm
- net Net-(SW9-B): track 81.8 -> 82.5 mm
- net Net-(U5-DEC3): track 65.0 -> 64.3 mm
- net C2-2: track 11.0 -> 11.5 mm
