File: hardware/mouse/rfradio.kicad_sch (KiCad schematic)
At the start: 19 parts, among them U5 nRF52840

Commit message: wowsa, thats a lot o' debugging
Parts:
- added J1: TC2050, Connector:Tag-Connect_TC2050-IDC-NL_2x05_P1.27mm_Vertical, symbol Connector:TC2050
Connections:
- net GND: now also J1.3
- net VBUS: now also J1.5
- net VDD_nRF: now also J1.1
- net SWDCLK: now reaches U5.AA24 (SWDCLK)
- net SWDCLK: now also J1.4
- net SWDIO: now reaches U5.AC24 (SWDIO)
- net SWDIO: now also J1.2
