File: hardware/mouse/mouse.kicad_pcb (KiCad board)
At the start: 6 copper layers, 44 x 68 mm, 83 parts, among them J1 TC2050, J2 JSTPH, J3 USB_C_Receptacle_USB2.0_14P, SW1 SW_SPST, SW2 SW_SPST, SW3 SW_SPST, SW4 SW_SPST, SW5 SW_SPST, SW6 SW_SPST, SW7 SW_SPST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

Commit message: some changes
Routing:
- net SWDCLK: track 0.00 -> 40.1 mm, vias 0 -> 2
- net SWDIO: track 0.00 -> 38.0 mm, vias 0 -> 2
- net VDDW1: track 105.1 -> 134.8 mm, vias 10 -> 11
- net VBUS: track 115.6 -> 120.2 mm, vias 8 -> 9
- net Net-(D3-K): track 55.3 -> 55.9 mm
