File: hardware/dongle/dongle/dongle.kicad_sch (KiCad schematic)
At the start: 0 parts

Commit message: trying to understand what jlc is doing
Parts:
- added 0.02, 0.29, 0.31, 1.10, 1.13, 1.15: ${ALTIUM_VALUE}, Castellated_Hole_0.9mm, symbol AltiumLib:root_1_TESTPAD_AltiumLib.DbLib
- added 0.04, 0.11, 0.26, GND4, VBUS2: ${ALTIUM_VALUE}, TP_SMD_D1.0mm, symbol AltiumLib:root_2_TESTPAD_AltiumLib.DbLib
- added 0.09, 0.10: ${ALTIUM_VALUE}, Castellated_Hole_0.9mm, symbol AltiumLib:root_0_TESTPAD_AltiumLib.DbLib
- added 0.13, 0.15, 0.17, 0.20, 0.22, 0.24, 1.00: ${ALTIUM_VALUE}, Castellated_Hole_0.9mm, symbol AltiumLib:root_3_TESTPAD_AltiumLib.DbLib
- added 0.14, D+, DP, UGND: ${ALTIUM_VALUE}, TP_SMD_D1.0mm, symbol AltiumLib:root_3_TESTPAD_AltiumLib.DbLib
- added 1.01, 1.02, 1.04, 1.07: ${ALTIUM_VALUE}, TP_SMD_D1.0mm, symbol AltiumLib:root_0_TESTPAD_AltiumLib.DbLib
- added 1.11, D-, DN: ${ALTIUM_VALUE}, TP_SMD_D1.0mm, symbol AltiumLib:root_1_TESTPAD_AltiumLib.DbLib
- added C1, C11, C2: ${ALTIUM_VALUE}, CAPC0603X03L_C, symbol AltiumLib:root_0_CAP_AltiumLib.DbLib
- added C12, C16, C5, C7, C8, C9: ${ALTIUM_VALUE}, CAPC0603X03L_C, symbol AltiumLib:root_3_CAP_AltiumLib.DbLib
- added C13, C25: ${ALTIUM_VALUE}, CAPC0603X03L_C_NC, symbol AltiumLib:root_3_CAP_AltiumLib.DbLib
- added C14, C20, C6: ${ALTIUM_VALUE}, CAPC1608X06L, symbol AltiumLib:root_3_CAP_AltiumLib.DbLib
- added C15: ${ALTIUM_VALUE}, CAPC1608X06L, symbol AltiumLib:root_1_CAP_AltiumLib.DbLib
- added C17, C18: ${ALTIUM_VALUE}, CAPC0603X03L_C, symbol AltiumLib:root_2_CAP_AltiumLib.DbLib
- added C19: ${ALTIUM_VALUE}, CAPC1005X04L, symbol AltiumLib:root_3_CAP_AltiumLib.DbLib
- added C21, C22, C24, C26, C27, C3, C4: ${ALTIUM_VALUE}, CAPC0603X03L_C, symbol AltiumLib:root_1_CAP_AltiumLib.DbLib
- added C23: ${ALTIUM_VALUE}, CAPC1005X04L, symbol AltiumLib:root_1_CAP_AltiumLib.DbLib
- added C28: ${ALTIUM_VALUE}, CAPC1005X04L_NC, symbol AltiumLib:root_1_CAP_AltiumLib.DbLib
- added C29: ${ALTIUM_VALUE}, CAPC1005X04L_NC, symbol AltiumLib:root_3_CAP_AltiumLib.DbLib
- added D1: ${ALTIUM_VALUE}, SOT190P230X110-4L, symbol AltiumLib:root_0_mirrored_PRTR5V0U2X_AltiumLib.DbLib
- added FB1, FB2: ${ALTIUM_VALUE}, INDC0603X03L_C, symbol AltiumLib:root_0_IND_F_AltiumLib.DbLib
- added Fid1: Fiducial mark, Fiducial_Square, symbol AltiumLib:root_0_Fiducial_AltiumLib.DbLib
- added Fid2: Fiducial mark, Fiducial, symbol AltiumLib:root_0_Fiducial_AltiumLib.DbLib
- added GND1, VBUS1: ${ALTIUM_VALUE}, Castellated_Hole_0.9mm, symbol AltiumLib:root_2_TESTPAD_AltiumLib.DbLib
- added GND2, GND3: ${ALTIUM_VALUE}, Castellated_Hole_0.9mm_S, symbol AltiumLib:root_2_TESTPAD_AltiumLib.DbLib
- added J1: ${ALTIUM_VALUE}, USB-A-PCB, symbol AltiumLib:root_0_USB-PCB-A_AltiumLib.DbLib
- added J2: ${ALTIUM_VALUE}, TC2050-IDC-NLFP, symbol AltiumLib:root_0_CONN-2x5_var2_No_BOM_AltiumLib.DbLib
- added L1: ${ALTIUM_VALUE}, INDC0603X03L_C, symbol AltiumLib:root_0_IND_AltiumLib.DbLib
- added L2: ${ALTIUM_VALUE}, INDC1608X06L, symbol AltiumLib:root_3_IND_AltiumLib.DbLib
- added L3: ${ALTIUM_VALUE}, INDC1005X04L, symbol AltiumLib:root_3_IND_AltiumLib.DbLib
- added L4: ${ALTIUM_VALUE}, INDC1608X06L, symbol AltiumLib:root_0_IND_AltiumLib.DbLib
- added LD1: ${ALTIUM_VALUE}, LED_0603_G, symbol AltiumLib:root_3_D{colon}LED_AltiumLib.DbLib
- added LD2: ${ALTIUM_VALUE}, LED_RGB_0603, symbol AltiumLib:root_0_D{colon}LED_RGB_AltiumLib.DbLib
- added P1: ${ALTIUM_VALUE}, HDR_2x5-SMD-1.27mm-NC, symbol AltiumLib:root_0_CONN-2x5_AltiumLib.DbLib
- added R1: ${ALTIUM_VALUE}, RESC0603X03L_C, symbol AltiumLib:root_0_RES_AltiumLib.DbLib
- added R2, R3, R4, R5, R6: ${ALTIUM_VALUE}, RESC0603X03L_C, symbol AltiumLib:root_1_RES_AltiumLib.DbLib
- added R7: ${ALTIUM_VALUE}, RESC0603X03L_C, symbol AltiumLib:root_2_RES_AltiumLib.DbLib
- added SB1: ${ALTIUM_VALUE}, Solderbridge, symbol AltiumLib:root_1_SOLDERBRIDGE_AltiumLib.DbLib
- added SB2, SB3, SB4: ${ALTIUM_VALUE}, Solderbridge_Shorted, symbol AltiumLib:root_0_SOLDERBRIDGE_SHORTED_AltiumLib.DbLib
- added SW1: ${ALTIUM_VALUE}, C&K_PTS810, symbol AltiumLib:root_3_SW-PB_AltiumLib.DbLib
- added SW2: ${ALTIUM_VALUE}, EVQP7A_J_B_K, symbol AltiumLib:root_3_SW-PB_AltiumLib.DbLib
- added SWDCLK, SWDIO: ${ALTIUM_VALUE}, Castellated_Hole_0.9mm_D, symbol AltiumLib:root_0_TESTPAD_AltiumLib.DbLib
- added U1: ${ALTIUM_VALUE}, AQFN50P700X700X85_HS-74N, symbol AltiumLib:root_0_nRF52840_QIAA_AltiumLib.DbLib
- added VDD OUT: ${ALTIUM_VALUE}, Castellated_Hole_0.9mm, symbol AltiumLib:root_2_TESTPAD_AltiumLib.DbLib
- added VDD nRF: ${ALTIUM_VALUE}, TP_SMD_D1.0mm, symbol AltiumLib:root_2_TESTPAD_AltiumLib.DbLib
- added X1: ${ALTIUM_VALUE}, BT-XTAL_2016, symbol AltiumLib:root_1_XTAL_4-pin_AltiumLib.DbLib
- added X2: ${ALTIUM_VALUE}, XTAL_2012, symbol AltiumLib:root_3_XTAL_2-pin_AltiumLib.DbLib
Connections:
- new net: C3.2, L1.1, U1.H23 (ANT)
- new net: D-.1, J1.2 (D-), SB3.2 (1)
- new net: LD1.1 (C), R3.2
- new net: D+.1, J1.3 (D+), SB4.2 (1)
- new net: FB2.1, J1.4 (GND), UGND.1
- new net: C1.2, X1.4 (GND)
- new net: LD2.3 (C_BLUE), R6.2
- new net: C20.1, U1.AC5 (DECUSB)
- new net: L2.1, L3.2
- new net: LD2.1 (C_RED), R4.2
- new net: LD2.2 (C_GREEN), R5.2
- new net: SB1.2 (1), SB2.1 (0), U1.Y2 (VDDH)
- new net: L2.2, U1.B3 (DCC)
- new net: C9.1, U1.N24 (DEC5)
- new net: L4.2, U1.AB2 (DCCH)
- new net: C13.1, U1.A18 (DEC2)
- new net ANT: C26.2, R1.2
- new net DEC1: C5.1, U1.C1 (DEC1)
- new net DEC3: C11.1, U1.D23 (DEC3)
- new net DEC4_6: C15.2, C16.1, L3.1, U1.B5 (DEC4), U1.E24 (DEC6)
- new net D_N: D1.2 (IO1), DN.1, SB3.1 (0), U1.AD4 (D-)
- new net D_P: D1.3 (IO2), DP.1, SB4.1 (0), U1.AD6 (D+)
- new net GND: C11.2, C12.2, C13.2, C14.2, C15.1, C16.2, C17.2, C18.2, C19.2, C2.2, C20.2, C21.1, C22.1, C23.1, C24.1, C25.2, C26.1, C27.1, C28.1, C29.2, C3.1, C4.1, C5.2, C6.2, C7.2, C8.2, C9.2, D1.1 (GND), FB2.2, GND1.1, GND2.1, GND3.1, GND4.1, J2.3, P1.3, P1.5, P1.9, SW1.2 (COM), SW2.2 (COM), U1.74 (GND), U1.B15 (P1.14), U1.B7 (VSS), U1.F23 (VSS_PA), X1.2 (GND)
- new net LED1: R3.1, U1.L1 (P0.06)
- new net LED2_B: R6.1, U1.U1 (P0.12)
- new net LED2_G: R5.1, U1.R1 (P1.09)
- new net LED2_R: R4.1, U1.N1 (P0.08)
- new net P0.00/XL1: C17.1, U1.D2 (P0.00/XL1), X2.1 (inp)
- new net P0.01/XL2: C18.1, U1.F2 (P0.01/XL2), X2.2 (out)
- new net P0.02: 0.02.1, U1.A12 (P0.02/AIN0)
- new net P0.04: 0.04.1, U1.J1 (P0.04/AIN2)
- new net P0.09: 0.09.1, C28.2, U1.L24 (P0.09/NFC1)
- new net P0.10: 0.10.1, C29.1, U1.J24 (P0.10/NFC2)
- new net P0.11: 0.11.1, U1.T2 (P0.11)
- new net P0.13: 0.13.1, U1.AD8 (P0.13)
- new net P0.14: 0.14.1, U1.AC9 (P0.14)
- new net P0.15: 0.15.1, U1.AD10 (P0.15)
- new net P0.17: 0.17.1, U1.AD12 (P0.17)
- new net P0.20: 0.20.1, U1.AD16 (P0.20)
- new net P0.22: 0.22.1, U1.AD18 (P0.22)
- new net P0.24: 0.24.1, U1.AD20 (P0.24)
- new net P0.26: 0.26.1, U1.G1 (P0.26)
- new net P0.29: 0.29.1, U1.A10 (P0.29/AIN5)
- new net P0.31: 0.31.1, U1.A8 (P0.31/AIN7)
- new net P1.00: 1.00.1, U1.AD22 (P1.00)
- new net P1.01: 1.01.1, U1.Y23 (P1.01)
- new net P1.02: 1.02.1, U1.W24 (P1.02)
- new net P1.04: 1.04.1, U1.U24 (P1.04)
- new net P1.07: 1.07.1, U1.P23 (P1.07)
- new net P1.10: 1.10.1, U1.A20 (P1.10)
- new net P1.11: 1.11.1, U1.B19 (P1.11)
- new net P1.13: 1.13.1, U1.A16 (P1.13)
- new net P1.15: 1.15.1, U1.A14 (P1.15)
- new net RESET: C27.2, P1.10, R2.1, SW2.1 (N.O), U1.AC13 (P0.18/RESET), U1.AC15 (P0.19), U1.AC17 (P0.21), U1.AC19 (P0.23), U1.AC21 (P0.25)
- new net RF: C25.1, C4.2, L1.2, R1.1
- new net SW1: SW1.1 (N.O), U1.R24 (P1.06)
- new net SWDCLK: J2.4, P1.4, SWDCLK.1, U1.AA24 (SWDCLK)
- new net SWDIO: J2.2, P1.2, SWDIO.1, U1.AC24 (SWDIO)
- new net VBUS: C22.2, FB1.2, R7.2
- new net VBUS': C21.2, C23.2, C24.2, D1.4 (VCC), FB1.1, J1.1 (VBUS), J2.5, VBUS1.1, VBUS2.1
- new net VBUS_nRF: C19.1, R7.1, SB2.2 (1), U1.AD2 (VBUS)
- new net VDD_nRF: C12.1, C14.1, C6.1, C7.1, C8.1, J2.1, L4.1, LD1.2 (A), LD2.4 (A), P1.1, R2.2, SB1.1 (0), U1.A22 (VDD), U1.AD14 (VDD), U1.AD23 (VDD), U1.B1 (VDD), U1.W1 (VDD), VDD OUT.1, VDD nRF.1
- new net XC1: C1.1, U1.B24 (XC1), X1.1 (IN)
- new net XC2: C2.1, U1.A23 (XC2), X1.3 (OUT)
- no-connect marks 0 -> 2
Other:
- note added: "${##}"
- note added: "${#}"
- note added: "${DRAWNBY}"
- note added: "${FILENAME}"
- note added: "${MODIFIEDDATE}"
- note added: "${PCANAME}"
- note added: "${REVISION}"
- note added: "${TITLE}"
- note added: "A4"
- note added: "Antenna"
- note added: "Date:"
- note added: "Drawn By:"
- note added: "File:"
- note added: "PCB Assembly Number"
- note added: "Revision"
- note added: "Sheet of"
- note added: "Size"
- note added: "Title"
- company: (none) -> Nordic Semiconductor
- title: (none) -> =BoardTitle
